File: adruino_0.kicad_pcb (KiCad board)
At the start: 2 copper layers, 67.1 x 57.4 mm, 21 parts, among them J1 Conn_01x04_Male, J10 Conn_01x04_Male, J11 Conn_02x02_Odd_Even, J12 Conn_01x02_Male, J13 locked, J14 Conn_02x14_Odd_Even, J15 Conn_01x04_Male, J16 Conn_02x02_Odd_Even, J2 Conn_01x04_Male, J3 Conn_01x04_Male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

Commit message: 基板更新
Parts:
- J13: value locked -> Conn_02x15_Odd_Even; footprint Connector_PinSocket_2.54mm:PinSocket_2x14_P2.54mm_Vertical -> Connector_PinHeader_2.54mm:PinHeader_2x15_P2.54mm_Vertical; moved to F.Cu
- J14: value Conn_02x14_Odd_Even -> Conn_02x15_Odd_Even; footprint Connector_PinSocket_2.54mm:PinSocket_2x14_P2.54mm_Vertical -> Connector_PinHeader_2.54mm:PinHeader_2x15_P2.54mm_Vertical; moved to F.Cu
- turned J14 to 0 degrees
- turned J13 to 0 degrees
Connections:
- J13 pad 23: +3.3V -> unconnected-(J13-Pad23)
- J13 pad 24: GND -> unconnected-(J13-Pad24)
- J13 pad 27: unconnected-(J13-Pad27) -> +3.3V
- J14 pad 23: +3.3V -> unconnected-(J14-Pad23)
- J14 pad 24: GND -> unconnected-(J14-Pad24)
Routing:
- net GND: track 340.5 -> 346.6 mm
- net +3.3V: track 258.9 -> 262.9 mm
Other:
- board size 67.1 x 57.4 mm -> 67.1 x 62.7 mm
- board text added: "Analog"
- board text added: "I2C"
- board text added: "UART"
- board text added: "fake UNO R4.0.1"
